Commit message: Update 12 Jul 23

File: lbr_description/urdf/med7/med7.urdf.xacro (robot description, xacro)
@@ -6,7 +6,8 @@
     <xacro:arg name="robot_name" default="lbr" />
     <xacro:arg name="sim" default="true" />
+    <xacro:arg name="world_name" default="world" />
     <!-- fix to world -->
-    <link name="world" />
+    <link name="$(arg world_name)" />
     <!-- med -->
-    <xacro:med7 parent="world" robot_name="$(arg robot_name)" sim="$(arg sim)" />
+    <xacro:med7 parent="$(arg world_name)" robot_name="$(arg robot_name)" sim="$(arg sim)" />
 </robot>
